Commit message: 2 drones but not working

File: sjtu_drone_description/urdf/sjtu_drone.urdf.xacro (robot description, xacro)
@@ -24,5 +24,5 @@
       <origin rpy="0 0 0" xyz="0   0   0.04"/>
       <geometry>
-        <mesh filename="file://$(find sjtu_drone_description)/models/sjtu_drone/quadrotor_4.stl"/>
+        <mesh filename="file://$(find sjtu_drone_description)/models/drone_1/quadrotor_4.stl"/>
         <!-- <mesh filename="package://sjtu_drone/quadrotor_4.stl"/> -->
       </geometry>
@@ -31,5 +31,5 @@
       <origin rpy="0 0 0" xyz="0   0   0.04"/>
       <geometry>
-        <mesh filename="file://$(find sjtu_drone_description)/models/sjtu_drone/quadrotor_4.dae"/>
+        <mesh filename="file://$(find sjtu_drone_description)/models/drone_1/quadrotor_4.dae"/>
         <!-- <mesh filename="package://sjtu_drone/quadrotor_4.dae"/> -->
       </geometry>
@@ -43,5 +43,5 @@
   <link name="front_cam_link"/>
   <gazebo>
-    <plugin name='simple_drone' filename='libplugin_drone.so'>
+    <plugin name='drone_1' filename='libplugin_drone.so'>
       <ros>
         <namespace>${mp['namespace']}</namespace>

File: sjtu_drone_description/urdf/sjtu_drone2.urdf.xacro (robot description, xacro)
@@ -24,5 +24,5 @@
       <origin rpy="0 0 0" xyz="0   0   0.04"/>
       <geometry>
-        <mesh filename="file://$(find sjtu_drone_description)/models/sjtu_drone/quadrotor_4.stl"/>
+        <mesh filename="file://$(find sjtu_drone_description)/models/drone_2/quadrotor_4.stl"/>
         <!-- <mesh filename="package://sjtu_drone/quadrotor_4.stl"/> -->
       </geometry>
@@ -31,5 +31,5 @@
       <origin rpy="0 0 0" xyz="0   0   0.04"/>
       <geometry>
-        <mesh filename="file://$(find sjtu_drone_description)/models/sjtu_drone/quadrotor_4.dae"/>
+        <mesh filename="file://$(find sjtu_drone_description)/models/drone_2/quadrotor_4.dae"/>
         <!-- <mesh filename="package://sjtu_drone/quadrotor_4.dae"/> -->
       </geometry>
@@ -43,5 +43,5 @@
   <link name="front_cam_link"/>
   <gazebo>
-    <plugin name='simple_drone' filename='libplugin_drone.so'>
+    <plugin name='drone_2' filename='libplugin_drone.so'>
       <ros>
         <namespace>${mp['namespace']}</namespace>

Commit message: problem with 2 drones

File: sjtu_drone_description/urdf/sjtu_drone.urdf.xacro (robot description, xacro)
@@ -25,5 +25,4 @@
       <geometry>
         <mesh filename="file://$(find sjtu_drone_description)/models/drone_1/quadrotor_4.stl"/>
-        <!-- <mesh filename="package://sjtu_drone/quadrotor_4.stl"/> -->
       </geometry>
     </collision>
@@ -32,5 +31,4 @@
       <geometry>
         <mesh filename="file://$(find sjtu_drone_description)/models/drone_1/quadrotor_4.dae"/>
-        <!-- <mesh filename="package://sjtu_drone/quadrotor_4.dae"/> -->
       </geometry>
     </visual>

File: sjtu_drone_description/urdf/sjtu_drone2.urdf.xacro (robot description, xacro)
@@ -25,5 +25,4 @@
       <geometry>
         <mesh filename="file://$(find sjtu_drone_description)/models/drone_2/quadrotor_4.stl"/>
-        <!-- <mesh filename="package://sjtu_drone/quadrotor_4.stl"/> -->
       </geometry>
     </collision>
@@ -32,5 +31,4 @@
       <geometry>
         <mesh filename="file://$(find sjtu_drone_description)/models/drone_2/quadrotor_4.dae"/>
-        <!-- <mesh filename="package://sjtu_drone/quadrotor_4.dae"/> -->
       </geometry>
     </visual>
