Commit message: Multiple drones rl tests works

File: sjtu_drone_description/urdf/multi_drone.urdf.xacro (robot description, xacro)
@@ -31,15 +31,9 @@
   </link>
   <joint name="${drone_id}/front_cam_joint" type="fixed">
-    <origin rpy="0 0.261799 0" xyz="0.2 0 0"/>
+    <origin rpy="0 0 0" xyz="0.2 0 0"/>
     <parent link="${drone_id}/base_link" />
     <child link="${drone_id}/front_cam_link" />
   </joint>
   <link name="${drone_id}/front_cam_link"/>
-  <joint name="${drone_id}/bottom_cam_joint" type="fixed">
-    <origin rpy="0 1.570796326794897 0" xyz="0 0 0"/>
-    <parent link="${drone_id}/base_link" />
-    <child link="${drone_id}/bottom_cam_link" />
-  </joint>
-  <link name="${drone_id}/bottom_cam_link"/>
   <gazebo>
     <plugin name='simple_drone' filename='libplugin_drone.so'>
@@ -56,9 +50,9 @@
       <velocityXYProportionalGain>5.0</velocityXYProportionalGain>
       <velocityXYDifferentialGain>2.3</velocityXYDifferentialGain>
-      <velocityXYLimit>2</velocityXYLimit>
+      <velocityXYLimit>30</velocityXYLimit>
       <velocityZProportionalGain>5.0</velocityZProportionalGain>
       <velocityZIntegralGain>0.0</velocityZIntegralGain>
       <velocityZDifferentialGain>1.0</velocityZDifferentialGain>
-      <velocityZLimit>-1</velocityZLimit>
+      <velocityZLimit>-30</velocityZLimit>
       <positionXYProportionalGain>1.1</positionXYProportionalGain>
       <positionXYDifferentialGain>0.0</positionXYDifferentialGain>
@@ -69,10 +63,43 @@
       <positionZIntegralGain>0.0</positionZIntegralGain>
       <positionZLimit>-1</positionZLimit>
-      <maxForce>30</maxForce>
+      <maxForce>300</maxForce>
       <motionSmallNoise>0.0</motionSmallNoise>
       <motionDriftNoise>0.0</motionDriftNoise>
-      <motionDriftNoiseTime>50.0</motionDriftNoiseTime>
+      <motionDriftNoiseTime>5.0</motionDriftNoiseTime>
     </plugin>
   </gazebo>
+  <!-- <gazebo>
+    <plugin name='simple_drone' filename='libplugin_drone.so'>
+      <bodyName>${drone_id}/base_link</bodyName>
+      <pub_odom>true</pub_odom>
+      <rosNamespace>${drone_id}</rosNamespace>
+      <imuTopic>${drone_id}/imu</imuTopic>
+      <rollpitchProportionalGain>10.0</rollpitchProportionalGain>
+      <rollpitchDifferentialGain>5.0</rollpitchDifferentialGain>
+      <rollpitchLimit>1.5</rollpitchLimit>
+      <yawProportionalGain>2.0</yawProportionalGain>
+      <yawDifferentialGain>1.0</yawDifferentialGain>
+      <yawLimit>20</yawLimit>
+      <velocityXYProportionalGain>5.0</velocityXYProportionalGain>
+      <velocityXYDifferentialGain>2.3</velocityXYDifferentialGain>
+      <velocityXYLimit>30</velocityXYLimit>
+      <velocityZProportionalGain>5.0</velocityZProportionalGain>
+      <velocityZIntegralGain>0.0</velocityZIntegralGain>
+      <velocityZDifferentialGain>1.0</velocityZDifferentialGain>
+      <velocityZLimit>30</velocityZLimit>
+      <positionXYProportionalGain>1.1</positionXYProportionalGain>
+      <positionXYDifferentialGain>0.0</positionXYDifferentialGain>
+      <positionXYIntegralGain>0.0</positionXYIntegralGain>
+      <positionXYLimit>5</positionXYLimit>
+      <positionZProportionalGain>1.0</positionZProportionalGain>
+      <positionZDifferentialGain>0.2</positionZDifferentialGain>
+      <positionZIntegralGain>0.0</positionZIntegralGain>
+      <positionZLimit>-1</positionZLimit>
+      <maxForce>300</maxForce>
+      <motionSmallNoise>0.05</motionSmallNoise>
+      <motionDriftNoise>0.03</motionDriftNoise>
+      <motionDriftNoiseTime>5.0</motionDriftNoiseTime>
+    </plugin>
+  </gazebo> -->
   <!-- Sensors -->
   <!-- IMU sensor in 100fps -->
@@ -101,5 +128,5 @@
         </ros>
         <initial_orientation_as_reference>false</initial_orientation_as_reference>
-        <frame_name>base_link</frame_name>
+        <frame_name>/${drone_id}/base_link</frame_name>
       </plugin>
     </sensor>
@@ -127,5 +154,5 @@
           <remapping>camera_info:=camera_front_info</remapping>
         </ros>
-        <frame_name>front_cam_link</frame_name>
+        <frame_name>/${drone_id}/front_cam_link</frame_name>
       </plugin>
     </sensor>
@@ -155,5 +182,5 @@
           <remapping>~/out:=~/nav</remapping>
         </ros>
-        <frame_name>base_link</frame_name>
+        <frame_name>/${drone_id}/base_link</frame_name>
       </plugin>
     </sensor>
